File: breadboard-inverter.kicad_pcb (KiCad board)
At the start: 2 copper layers, 14.2 x 49.8 mm, 13 parts, among them J1 Conn_02x01, J2 Conn_02x01, J3 Conn_02x01, J4 Conn_02x01, J5 Conn_01x04, J6 Conn_01x04, U1 TL072

Commit message: Add image and schematic
Parts:
- removed J3, J4: Conn_02x01, Connector_PinHeader_2.54mm:PinHeader_2x01_P2.54mm_Vertical
- J1, J2: value Conn_02x01 -> Conn_02x05; footprint Connector_PinHeader_2.54mm:PinHeader_2x01_P2.54mm_Vertical -> Connector_PinHeader_2.54mm:PinHeader_2x05_P2.54mm_Vertical
- moved J1 10.2 mm to (142.2, 61.0)
- moved J2 2.54 mm to (132.1, 109.2)
- moved C2 1.99 mm to (141.0, 97.5)
- moved J5 1.99 mm to (133.3, 100.8)
- moved R2 1.99 mm to (136.9, 100.8)
- moved R1 1.99 mm to (137.2, 93.2)
- moved U1 1.27 mm to (133.4, 88.9)
Routing:
- net GND: track 105.6 -> 102.4 mm
- net Net-(R3-Pad1): track 10.9 -> 12.1 mm
- net Net-(J6-Pad3): track 11.8 -> 13.1 mm
- net +12V: track 31.0 -> 32.3 mm
- net -12V: track 31.0 -> 32.2 mm
- net Net-(J5-Pad3): track 10.6 -> 11.6 mm
- net Net-(R1-Pad1): track 12.6 -> 13.4 mm
Other:
- board size 14.2 x 49.8 mm -> 14.2 x 52.3 mm
- board text added: "IN"
- board text added: "OUT"
