File: breadboard-inverter.kicad_sch (KiCad schematic)
At the start: 13 parts, among them J2 Conn_02x01, J3 Conn_02x01, J4 Conn_02x01, J6 Conn_01x04

Commit message: Add image and schematic
Parts:
- removed J3, J4: Conn_02x01, symbol Connector_Generic:Conn_02x01
- C1, C2: value (none) -> 100nF; footprint (none) -> Capacitor_THT:C_Disc_D4.7mm_W2.5mm_P5.00mm
- J1: value (none) -> Conn_02x05; footprint (none) -> Connector_PinHeader_2.54mm:PinHeader_2x05_P2.54mm_Vertical; symbol Connector_Generic:Conn_02x01 -> Connector_Generic:Conn_02x05_Odd_Even
- J2: value Conn_02x01 -> Conn_02x05; footprint (none) -> Connector_PinHeader_2.54mm:PinHeader_2x05_P2.54mm_Vertical; symbol Connector_Generic:Conn_02x01 -> Connector_Generic:Conn_02x05_Odd_Even
- J5: value (none) -> Conn_01x04; footprint (none) -> Connector_PinHeader_2.54mm:PinHeader_1x04_P2.54mm_Vertical
- J6: footprint (none) -> Connector_PinHeader_2.54mm:PinHeader_1x04_P2.54mm_Vertical
- R1, R2, R3, R4: value (none) -> 100k; footprint (none) -> Resistor_THT:R_Axial_DIN0207_L6.3mm_D2.5mm_P2.54mm_Vertical
- U1: value (none) -> TL072; footprint (none) -> Package_DIP:DIP-8_W7.62mm_Socket
Connections:
- net +12V: now also J1.3 (Pin_3), J1.5 (Pin_5), J1.7 (Pin_7), J1.9 (Pin_9)
- net -12V: now also J2.3 (Pin_3), J2.5 (Pin_5), J2.7 (Pin_7), J2.9 (Pin_9)
- net GND: now also J1.10 (Pin_10), J1.4 (Pin_4), J1.6 (Pin_6), J1.8 (Pin_8), J2.10 (Pin_10), J2.4 (Pin_4), J2.6 (Pin_6), J2.8 (Pin_8)
Other:
- moved on the sheet: C1, C2, J5, J6, R1, R2, R3, R4, U1A, U1B, U1C
